File: BW1098OBC_Power_Supply-SchDoc.sch (KiCad schematic (older format))
At the start: 80 parts, among them J7 PJ-050AH or NEB21R, J8 B2B-PH-K-S(LF)(SN), U1 TLV70733PDQN, U2 TLV70018DCK, U3 TLV70028DCK, U4 TLV62080DSG, U8 TLV70012DCK

Commit message: Update
Parts:
- removed 1V05_2, 1V05_3: 1V05, symbol power:GND
- removed 1V2_2, 1V2_3: 1V2, symbol power:GND
- removed 1V8_3, 1V8_4: 1V8, symbol power:GND
- removed 2V8_3, 2V8_4: 2V8, symbol power:GND
- removed 3V3, 3V3_2: 3V3, symbol power:GND
- removed C13, C14, C22: 22uF 0603, symbol BW1098OBC_Power_Supply-SchDoc-rescue:GRM188R61A226ME15D-
- removed C15, C17, C18, C19, C20, C21, C38, C39: 10uF 0603, symbol BW1098OBC_Power_Supply-SchDoc-rescue:GRM188R61A106ME69D-
- removed C16: 1uF 0402, symbol BW1098OBC_Power_Supply-SchDoc-rescue:GRM155R61E105KA12D-
- removed GND_33, GND_34, GND_35, GND_36, GND_37, GND_38, GND_39, GND_40, GND_41, GND_42, GND_43, GND_44, GND_45, GND_46, GND_47, GND_48, GND_49, GND_50, GND_51, GND_52, GND_53, GND_54, GND_55, GND_56: GND, symbol power:GND
- removed J7: PJ-050AH or NEB21R, symbol BW1098OBC_Power_Supply-SchDoc-rescue:PJ-050AH_NEB21R_COMBO-
- removed J8: B2B-PH-K-S(LF)(SN), symbol BW1098OBC_Power_Supply-SchDoc-rescue:B2B-PH-K-S(LF)(SN)-
- removed L1: 1uH, 3.2A, 20%, symbol BW1098OBC_Power_Supply-SchDoc-rescue:DFE252012P-1R0M=P2-
- removed R5, R6: 0R 0603, symbol BW1098OBC_Power_Supply-SchDoc-rescue:CRCW06030000Z0EA-
- removed R7: 53.6k 0402, symbol BW1098OBC_Power_Supply-SchDoc-rescue:CRCW040253K6FKED-
- removed R8: 39.2k 0402, symbol BW1098OBC_Power_Supply-SchDoc-rescue:CRCW040239K2FKED-
- removed TP10, TP11, TP12, TP13, TP14, TP15, TP16, TP17, TP6, TP7, TP8, TP9: (no value), symbol BW1098OBC_Power_Supply-SchDoc-rescue:TEST_POINT-
- removed U1: TLV70733PDQN, symbol BW1098OBC_Power_Supply-SchDoc-rescue:TLV70733PDQN-
- removed U2: TLV70018DCK, symbol BW1098OBC_Power_Supply-SchDoc-rescue:TLV70018DCK-
- removed U3: TLV70028DCK, symbol BW1098OBC_Power_Supply-SchDoc-rescue:TLV70028DCK-
- removed U4: TLV62080DSG, symbol BW1098OBC_Power_Supply-SchDoc-rescue:TLV62080DSG-
- removed U8: TLV70012DCK, symbol BW1098OBC_Power_Supply-SchDoc-rescue:TLV70012DCK-
- removed VBUS_3, VBUS_4: VBUS, symbol power:GND
- removed VDD_5V_10, VDD_5V_11, VDD_5V_12, VDD_5V_13, VDD_5V_14, VDD_5V_15, VDD_5V_16, VDD_5V_9: VDD_5V, symbol power:GND
Connections:
- net labels removed: 1. AVDD rising can occur before or after DOVDD rising as long as they are rising before XSHUTDOWN rising  2. XSHUTDOWN is pulled up after AVDD and DOVDD are stable  3. DVDD rises after DOVDD, but before XSHUTDOWN is pulled high, 10V, 1V05, 1V2, 1V8, 25V, 2V8, 3V3, GND, POWER SEQUENCING REQUIREMENTS:    The BW1099 module handles it's own power sequencing on-board.     The camera modules have their own power sequencing requirements. The OV9282 have requirements for sequencing, and the IMX378 has a max slew rate requirement. See above., Parameter Set, Power_trace, VBUS, VDD_5V
- wire segments 89 -> 0
- no-connect marks 4 -> 0
Other:
- note removed: "(VANA, VIF, VDIG)"
- note removed: "*"
- note removed: "0V"
- note removed: "1.05V"
- note removed: "1.05V ± 0.1"
- note removed: "1.2V"
- note removed: "1.8V"
- note removed: "1.8V ± 0.1"
- note removed: "1925 Harmony Park Drive"
- note removed: "2.5mA"
- note removed: "2.8V"
- note removed: "2.8V ± 0.1"
- note removed: "24mA"
- note removed: "3.3V USB SW POWER"
- note removed: "446mA"
- note removed: "5"
- note removed: "52mA"
- note removed: "55mA"
- note removed: "8"
- note removed: "80234"
- note removed: "=document_number"
- note removed: "=drawn_by"
- note removed: "=project_title"
- note removed: "=revision"
- note removed: "AVDD"
- note removed: "DOVDD"
- note removed: "DVDD"
- note removed: "Date:"
- note removed: "Drawn by:"
- note removed: "FAN CONTROLLER"
- note removed: "Hardware Standby"
- note removed: "IMX378 POWER REQUIREMENTS"
- note removed: "IOUT= 1200mA"
- note removed: "IOUT= 300mA"
- note removed: "Luxonis Holding"
- note removed: "Max Current"
- note removed: "Max Slew Rate: 50 mV/µs"
- note removed: "Module"
- note removed: "No power supply sequencing is needed"
- note removed: "Number:"
- note removed: "OV9282 POWER REQUIREMENTS"
- note removed: "POWER INPUT"
- note removed: "POWER SUPPLIES FOR CAMERA MODULES"
- note removed: "Power OFF"
- note removed: "Revision:"
- note removed: "Sensor"
- note removed: "Sheet"
- note removed: "Size:"
- note removed: "Slew Rate Constraint"
- note removed: "Slew Rate: 18 mV/µs"
- note removed: "Slew Rate: 28 mV/µs"
- note removed: "Supply Information"
- note removed: "Supply Name"
- note removed: "Tabloid"
- note removed: "Time:"
- note removed: "Title"
- note removed: "United States"
- note removed: "VANA"
- note removed: "VDD"
- note removed: "VDD-A"
- note removed: "VDD-D"
- note removed: "VDD-IO"
- note removed: "VDIG"
- note removed: "VIF"
- note removed: "VOUT= 0.45x(R2+R3)/R3"
- note removed: "VOUT= 1.065V"
- note removed: "VOUT= 1.2V"
- note removed: "VOUT= 1.8V"
- note removed: "VOUT= 2.8V"
- note removed: "Voltage"
- note removed: "Westminster, CO"
- note removed: "XSHUTDOWN"
- note removed: "min 0ms"
- note removed: "min 1ms"
- note removed: "of"
