File: BW1098OBC_Power_Supply.sch (KiCad schematic (older format))
At the start: 80 parts

Commit message: More deletion of corrupted or duplicate files, added footprints and associations for mounting holes and 30 pin connector
Parts:
- removed 1V05_? (x2): 1V05, symbol power:GND
- removed 1V2_? (x2): 1V2, symbol power:GND
- removed 1V8_? (x2): 1V8, symbol power:GND
- removed 2V8_? (x2): 2V8, symbol power:GND
- removed 3V3_?, 3V?: 3V3, symbol power:GND
- removed GND_? (x24): GND, symbol power:GND
- removed VBUS_? (x2): VBUS, symbol power:GND
- removed VDD_5V_? (x8): VDD_5V, symbol power:GND
- gave numbers to parts that had none: 36
