File: BW1098OBC_TopLevel.sch (KiCad schematic (older format))
At the start: 6 parts

Commit message: Update
Changed lines of the file:
@@
 Text HLabel 2000 1700 0    60   Output ~ 0
 1V05
-$Sheet
-S 500  1000 1500 1000
-U 5FD7EFCB
-F0 "U_BW1098OBC_Power_Supply" 60
-F1 "BW1098OBC_Power_Supply-SchDoc.sch" 60
-$EndSheet
 Text HLabel 13600 4700 2    60   BiDi ~ 0
 MIPI_CAM_B
@@
 Text HLabel 13600 5100 2    60   Output ~ 0
 COM_AUX_IO2
-$Sheet
-S 13600 2800 1500 4800
-U 5FD7EFCD
-F0 "U_BW1098OBC_Connector" 60
-F1 "BW1098OBC_Connector-SchDoc.sch" 60
-$EndSheet
 Text HLabel 6800 3100 2    60   Input ~ 0
 2V8
@@
 Text HLabel 6800 3200 2    60   Input ~ 0
 1V8
-$Sheet
-S 6800 3000 1500 800
-U 5FD7EFCF
-F0 "U_BW1098OBC_IMX378" 60
-F1 "BW1098OBC_IMX378-SchDoc.sch" 60
-$EndSheet
 Text HLabel 8300 6500 0    60   BiDi ~ 0
 MIPI_CAM_C
@@
 Text HLabel 8300 6600 0    60   BiDi ~ 0
 CTL_CAM_B
-$Sheet
-S 6800 6300 1500 1100
-U 5FD7EFD1
-F0 "U_BW1098OBC_RIGHT_OV9282" 60
-F1 "BW1098OBC_RIGHT_OV9282-SchDoc.sch" 60
-$EndSheet
 Text HLabel 8300 4900 0    60   BiDi ~ 0
 I2C2
@@
 Text HLabel 8300 5100 0    60   Input ~ 0
 COM_AUX_IO2
-$Sheet
-S 6800 4500 1500 1100
-U 5FD7EFD3
-F0 "U_BW1098OBC_LEFT_OV9282" 60
-F1 "BW1098OBC_LEFT_OV9282-SchDoc.sch" 60
-$EndSheet
 $Comp
 L power:GND GND_66
@@
 Text HLabel 10300 5600 2    60   Input ~ 0
 VDD_5V
-$Sheet
-S 10300 5500 1500 400
-U 5FD7F014
-F0 "U_BW1098OBC_USB" 60
-F1 "BW1098OBC_USB-SchDoc.sch" 60
-$EndSheet
-$Sheet
-S 1000 9400 2000 600
-U 5FD7F01D
-F0 "U_BW1098OBC_Project_Information" 60
-F1 "BW1098OBC_Project_Information-SchDoc.sch" 60
-$EndSheet
 Wire Wire Line
 	3000 1600 2000 1600
@@
 Text Notes 12700 10000 0    50   ~ 0
 8
+$Sheet
+S 6800 6300 1500 1100
+U 5FD7EFD1
+F0 "U_BW1098OBC_RIGHT_OV9282" 60
+F1 "BW1098OBC_RIGHT_OV9282.sch" 60
+$EndSheet
+$Sheet
+S 6800 4500 1500 1100
+U 5FD7EFD3
+F0 "U_BW1098OBC_LEFT_OV9282" 60
+F1 "BW1098OBC_LEFT_OV9282.sch" 60
+$EndSheet
+$Sheet
+S 6800 3000 1500 800
+U 5FD7EFCF
+F0 "U_BW1098OBC_IMX378" 60
+F1 "BW1098OBC_IMX378.sch" 60
+$EndSheet
+$Sheet
+S 10300 5500 1500 400
+U 5FD7F014
+F0 "U_BW1098OBC_USB" 60
+F1 "BW1098OBC_USB.sch" 60
+$EndSheet
+$Sheet
+S 13600 2800 1500 4800
+U 5FD7EFCD
+F0 "U_BW1098OBC_Connector" 60
+F1 "BW1098OBC_Connector.sch" 60
+$EndSheet
+$Sheet
+S 1000 9400 2000 600
+U 5FD7F01D
+F0 "U_BW1098OBC_Project_Information" 60
+F1 "BW1098OBC_Project_Information.sch" 60
+$EndSheet
+$Sheet
+S 500  1000 1500 1000
+U 5FD7EFCB
+F0 "U_BW1098OBC_Power_Supply" 60
+F1 "BW1098OBC_Power_Supply.sch" 60
+$EndSheet
 $EndSCHEMATC

Commit message: More deletion of corrupted or duplicate files, added footprints and associations for mounting holes and 30 pin connector
Parts:
- removed GND_66, GND_67, GND_68, GND_? (x3): GND, symbol power:GND
Changed lines of the file:
@@
 COM_AUX_IO2
 $Comp
-L power:GND GND_66
+L power:GND #GND_066
 U 1 1 5FD7E7BA
 P 8300 3700
-F 0 "GND_66" H 8300 3550 20  0001 C CNN
+F 0 "#GND_066" H 8300 3550 20  0001 C CNN
 F 1 "GND" H 8250 3550 30  0000 C CNN
 F 2 "" H 8300 3700 70  0000 C CNN
@@
 $EndComp
 $Comp
-L power:GND GND_68
+L power:GND #GND_068
 U 1 1 5FD7E7B8
 P 2000 1900
-F 0 "GND_68" H 1950 1700 20  0001 C CNN
+F 0 "#GND_068" H 1950 1700 20  0001 C CNN
 F 1 "GND" H 1950 1800 30  0000 C CNN
 F 2 "" H 2000 1900 70  0000 C CNN
@@
 Connection ~ 10100 2900
 $Comp
-L power:GND GND_67
+L power:GND #GND_067
 U 1 1 5FD7E7B9
 P 8300 5500
-F 0 "GND_67" H 8300 5500 20  0001 C CNN
+F 0 "#GND_067" H 8300 5500 20  0001 C CNN
 F 1 "GND" H 8300 5430 30  0000 C CNN
 F 2 "" H 8300 5500 70  0000 C CNN
@@
 $EndComp
 $Comp
-L power:GND GND_?
+L power:GND #GND_0101
 U 1 1 5FD8846F
 P 11800 5800
-F 0 "GND_?" H 11800 5800 20  0001 C CNN
+F 0 "#GND_0101" H 11800 5800 20  0001 C CNN
 F 1 "GND" H 11800 5730 30  0000 C CNN
 F 2 "" H 11800 5800 70  0000 C CNN
@@
 $EndComp
 $Comp
-L power:GND GND_?
+L power:GND #GND_0102
 U 1 1 5FD89034
 P 15100 7500
-F 0 "GND_?" H 15100 7500 20  0001 C CNN
+F 0 "#GND_0102" H 15100 7500 20  0001 C CNN
 F 1 "GND" H 15100 7430 30  0000 C CNN
 F 2 "" H 15100 7500 70  0000 C CNN
@@
 $EndComp
 $Comp
-L power:GND GND_?
+L power:GND #GND_0103
 U 1 1 5FD8D529
 P 8300 7300
-F 0 "GND_?" H 8300 7300 20  0001 C CNN
+F 0 "#GND_0103" H 8300 7300 20  0001 C CNN
 F 1 "GND" H 8300 7230 30  0000 C CNN
 F 2 "" H 8300 7300 70  0000 C CNN
